File: Boards/Board-Version2/board2.brd (EAGLE design)
At the start: 127 x 101.6 mm, 9 parts

Commit message: i did a naughty Owo~
Parts:
- moved U$4 6.84 mm to (114.3, 6.35), turned to 90 degrees
- moved U$5 5.68 mm to (12.7, 6.35), turned to 270 degrees
Routing:
- net GND: track 332.1 -> 355.7 mm
- net +5V: track 224.3 -> 242.5 mm
- net N$47: track 118.9 -> 108.3 mm
- net N$65: track 112.3 -> 105.6 mm
- net N$32: track 106.1 -> 99.4 mm
- net N$63: track 95.4 -> 99.6 mm
- net N$22: track 109.6 -> 105.7 mm
- net N$62: track 115.9 -> 112.1 mm
- net N$12: track 97.5 -> 95.9 mm
- net N$48: track 107.4 -> 108.5 mm
- net N$64: track 103.8 -> 102.7 mm
